Commit message: cleaning up

File: robotics/ros/catkin_ws/src/r2d2/model.xacro (robot description, xacro)
@@ -1,7 +1,7 @@
 <?xml version="1.0" ?>
-<robot name="mrm" xmlns:xacro="http://www.ros.org/wiki/xacro">
+<robot name="r2d2">
     <link name="base_link">
         <visual>
-            <origin rpy="0 0 0" xyz="0 0 0"/>
+            <origin rpy="0 0 0" xyz="0 0 0.25"/>
             <geometry>
                 <box size=".5 .5 .5"/>
@@ -9,5 +9,5 @@
         </visual>
     </link>
-    <joint name="base_link__link_01" type="revolute">
+    <joint name="joint1" type="revolute">
         <axis xyz="0 0 1" />
         <limit effort="1000.0" lower="-3.14" upper="3.14" velocity="0.5" />
@@ -18,7 +18,61 @@
     <link name="link1">
         <visual>
-            <origin rpy="0 0 0" xyz="0 0 0.2"/>
+            <origin rpy="0 0 0" xyz="0 0 0.1"/>
             <geometry>
-                <box size="0.2 1 0.2"/>
+                <cylinder radius="0.2" length="0.2"/>
+            </geometry>
+        </visual>
+    </link>
+    <joint name="link_01_link_02" type="fixed">
+        <origin xyz="0 0 0"/>
+        <parent link="link1"/>
+        <child link="link2"/>
+    </joint>
+    <link name="link2">
+        <visual>
+            <origin rpy="0 0 0" xyz="0 0.5 0.1"/>
+            <geometry>
+                <box size=".2 1 .2"/>
+            </geometry>
+        </visual>
+    </link>
+    <joint name="link_02_link_03" type="fixed">
+        <origin xyz="0 0 0"/>
+        <parent link="link2"/>
+        <child link="link3"/>
+    </joint>
+    <link name="link3">
+        <visual>
+            <origin rpy="0 1.5708 0" xyz="0 1 0.1"/>
+            <geometry>
+                <cylinder radius="0.2" length="0.2"/>
+            </geometry>
+        </visual>
+    </link>
+    <joint name="joint2" type="revolute">
+        <axis xyz="1 0 0" />
+        <limit effort="1000.0" lower="-3.14" upper="3.14" velocity="0.5" />
+        <origin rpy="0 0 0" xyz="0 1 0.1"/>
+        <parent link="link3"/>
+        <child link="link4"/>
+    </joint>
+    <link name="link4">
+        <visual>
+            <origin rpy="0 1.5708 0" xyz="0 0 0"/>
+            <geometry>
+                <cylinder radius="0.2" length="0.2"/>
+            </geometry>
+        </visual>
+    </link>
+    <joint name="link_04_link_05" type="fixed">
+        <origin xyz="0 0 0"/>
+        <parent link="link4"/>
+        <child link="link5"/>
+    </joint>
+    <link name="link5">
+        <visual>
+            <origin rpy="0 0 0" xyz="0 0.5 0"/>
+            <geometry>
+                <box size=".2 1 .2"/>
             </geometry>
         </visual>
