Commit message: report almost done. Need to write the validation part

File: robotics/ros/assignment_ws/src/basic_robot/model/model.xacro (robot description, xacro)
@@ -1,5 +1,11 @@
 <?xml version="1.0" ?>
 <robot name="r2d2" xmlns:xacro="http://www.ros.org/wiki/xacro">
-    <link name="base_link">
+	<material name="blue">
+		<color rgba="0 0 0.8 1"/>
+    </material>
+    <material name="white">
+		<color rgba="1 1 1 1"/>
+    </material>
+    <link name="base">
         <visual>
             <origin rpy="0 0 0" xyz="0 0 0.25"/>
@@ -7,14 +13,15 @@
                 <box size=".1 .1 .5"/>
             </geometry>
+			<material name="white"/>
         </visual>
     </link>
-    <joint name="joint1" type="revolute">
+    <joint name="lowerJoint" type="revolute">
         <axis xyz="0 0 1" />
         <limit effort="1000.0" lower="-3.14" upper="3.14" velocity="0.5" />
         <origin rpy="0 0 0" xyz="0 0 0.5"/>
-        <parent link="base_link"/>
-        <child link="link1"/>
+        <parent link="base"/>
+        <child link="lowerLink"/>
     </joint>
-    <link name="link1">
+    <link name="lowerLink">
         <visual>
             <origin rpy="0 0 0" xyz="0 0 0.1"/>
@@ -22,14 +29,15 @@
                 <cylinder radius="0.12" length="0.2"/>
             </geometry>
+			<material name="blue"/>
         </visual>
     </link>
-    <joint name="joint2" type="revolute">
+    <joint name="upperJoint" type="revolute">
         <axis xyz="1 0 0" />
         <limit effort="1000.0" lower="-3.14" upper="3.14" velocity="0.5" />
         <origin rpy="0 0 0" xyz="0 0 0.1"/>
-        <parent link="link1"/>
-        <child link="link2"/>
+        <parent link="lowerLink"/>
+        <child link="upperLink"/>
     </joint>
-    <link name="link2">
+    <link name="upperLink">
         <visual>
             <origin rpy="0 0 0" xyz="0 0.5 0"/>
@@ -37,4 +45,5 @@
                 <box size=".1 1 .1"/>
             </geometry>
+			<material name="white"/>
         </visual>
     </link>
